Commit message: Changes in agv2_controller.py

File: models/agv_macros.xacro (robot description, xacro)
@@ -25,12 +25,13 @@
                 <surface>
                     <friction>
-                        <kp>1000000.0</kp> <!-- kp and kd for rubber -->
-                        <kd>100.0</kd>
-                        <mu>1.0</mu>
-                        <mu2>1.0</mu2>
-                        <slip1>0.5</slip1>
+                        <kp>10000000.0</kp> <!-- kp and kd for rubber -->
+                        <kd>1.0</kd>
+                        <mu>1.0</mu>    <!-- Coulomb friction mus-->
+                        <mu2>1.0</mu2>  <!-- Friction coefficient muk-->
+                        <fdir1>1 0 0</fdir1>
+                        <slip1>0.0</slip1>
                         <slip2>0.0</slip2>
                         <maxVel>1.0</maxVel>
-                        <minDepth>0.00</minDepth>
+                        <minDepth>0.001</minDepth>
                     </friction>
                 </surface>

File: models/agv_model.urdf.xacro (robot description, xacro)
@@ -9,5 +9,5 @@
     <xacro:property name="chasis_length" value="${scale * 0.5}" />
     <xacro:property name="chasis_height" value="${scale * 0.3}" />
-    <xacro:property name="chasis_mass" value="${scale * 50}" />
+    <xacro:property name="chasis_mass" value="${scale * 25}" />
     <xacro:property name="base_x_offset" value="0.0" />
     <xacro:property name="chasis_x_pos" value="${base_x_offset/1.0}" />
@@ -22,13 +22,13 @@
     <xacro:property name="chasis_inertia_zz" value="${chasis_mass/12.0 * (width_2 + length_2)}" />
     <xacro:property name="chasis_frame_width" value="${chasis_width - 2.1 * wheel_length}" />
-    <xacro:property name="chasis_frame_length" value="${chasis_length*1.2}" />
-    <xacro:property name="chasis_frame_height" value="${chasis_height/4.0}" />
-    <xacro:property name="hardware_width" value="${chasis_frame_width/1.0}" />
+    <xacro:property name="chasis_frame_length" value="${chasis_length * 1.2}" />
+    <xacro:property name="chasis_frame_height" value="${chasis_height / 4.0}" />
+    <xacro:property name="hardware_width" value="${chasis_frame_width / 1.0}" />
     <xacro:property name="hardware_length" value="${0.15}" />
-    <xacro:property name="hardware_height" value="${chasis_height/2.5}" />
-    <xacro:property name="hardware_z_offset" value="${hardware_height/2.0}" />
+    <xacro:property name="hardware_height" value="${chasis_height / 2.5}" />
+    <xacro:property name="hardware_z_offset" value="${hardware_height / 2.0}" />
     <xacro:property name="hardware_x_offset" value="${base_x_offset + (chasis_length/2.0) - (hardware_length/8.5)}" />
     <xacro:property name="hardware_length_back" value="${0.1}" />
-    <xacro:property name="hardware_height_2" value="${chasis_height/1.8}" />
+    <xacro:property name="hardware_height_2" value="${chasis_height / 1.8}" />
     <xacro:property name="hardware_z_offset_2" value="${hardware_height_2/2.0}" />
     <xacro:property name="hardware_minx_offset" value="${base_x_offset + -1.0*(chasis_length/2.0) - (hardware_length_back/8.5)}" />

File: models/agv_model_three.urdf.xacro (robot description, xacro)
@@ -9,5 +9,5 @@
     <xacro:property name="chasis_length" value="${scale * 0.5}" />
     <xacro:property name="chasis_height" value="${scale * 0.3}" />
-    <xacro:property name="chasis_mass" value="${scale * 50}" />
+    <xacro:property name="chasis_mass" value="${scale * 25}" />
     <xacro:property name="base_x_offset" value="0.0" />
     <xacro:property name="chasis_x_pos" value="${base_x_offset/1.0}" />

File: models/agv_model_two.urdf.xacro (robot description, xacro)
@@ -9,5 +9,5 @@
     <xacro:property name="chasis_length" value="${scale * 0.5}" />
     <xacro:property name="chasis_height" value="${scale * 0.3}" />
-    <xacro:property name="chasis_mass" value="${scale * 50}" />
+    <xacro:property name="chasis_mass" value="${scale * 25}" />
     <xacro:property name="base_x_offset" value="0.0" />
     <xacro:property name="chasis_x_pos" value="${base_x_offset/1.0}" />

Commit message: Add more Tags Modify the multi robots launch file

File: models/agv_macros.xacro (robot description, xacro)
@@ -25,12 +25,12 @@
                 <surface>
                     <friction>
-                        <kp>10000000.0</kp> <!-- kp and kd for rubber -->
+                        <kp>1000000.0</kp> <!-- kp and kd for rubber -->
                         <kd>1.0</kd>
-                        <mu>1.0</mu>    <!-- Coulomb friction mus-->
+                        <mu1>1.0</mu1>    <!-- Coulomb friction mus-->
                         <mu2>1.0</mu2>  <!-- Friction coefficient muk-->
                         <fdir1>1 0 0</fdir1>
                         <slip1>0.0</slip1>
                         <slip2>0.0</slip2>
-                        <maxVel>1.0</maxVel>
+                        <maxVel>10.0</maxVel>
                         <minDepth>0.001</minDepth>
                     </friction>
@@ -43,18 +43,7 @@
             <parent link="${parent}"/>
             <axis xyz="0 1 0" rpy="0 0 0"/>
-            <limit effort="10000" velocity="5.0"/>
-            <joint_properties damping="1.0" friction="1.0"/>
+            <limit effort="100" velocity="5.0"/>
+            <joint_properties damping="0.7"/>
         </joint>
     </xacro:macro>
-    <!-- ************************ Create joints for wheels ************************ -->
-    <!-- <xacro:macro name="jointz" params="name parent child origin_xyz">
-        <joint name="${name}" type="continuous">
-            <origin xyz="${origin_xyz}" rpy="0 0 0" />
-            <child link="${child}"/>
-            <parent link="${parent}"/>
-            <axis xyz="0 1 0" rpy="0 0 0"/>
-            <limit effort="10000" velocity="5.0"/>
-            <joint_properties damping="1.0" friction="1.0"/>
-        </joint>
-    </xacro:macro> -->
 </robot>

File: models/agv_model.urdf.xacro (robot description, xacro)
@@ -9,5 +9,5 @@
     <xacro:property name="chasis_length" value="${scale * 0.5}" />
     <xacro:property name="chasis_height" value="${scale * 0.3}" />
-    <xacro:property name="chasis_mass" value="${scale * 25}" />
+    <xacro:property name="chasis_mass" value="${scale * 150}" />
     <xacro:property name="base_x_offset" value="0.0" />
     <xacro:property name="chasis_x_pos" value="${base_x_offset/1.0}" />
@@ -37,5 +37,5 @@
     <xacro:property name="wheel_length" value="${scale * 0.05}" />
     <xacro:property name="wheel_radius" value="${scale * 0.08}" />
-    <xacro:property name="wheel_mass" value="${scale * 1.5}" />
+    <xacro:property name="wheel_mass" value="${scale * 2.637}" />
     <xacro:property name="wheel_x_offset" value="${base_x_offset + chasis_length/2.0}" />
     <xacro:property name="wheel_y_offset" value="${chasis_width/2.0 - wheel_length/2.0}" />
@@ -126,5 +126,5 @@
             <origin xyz="${artag_x_pos} 0 ${hardware_z_offset}" rpy="-1.5707 0 1.5707" />
             <geometry>
-                <box size="0.2 0.2 0.01"/>
+                <mesh filename="package://tec_proyect/meshes/aruco_id0.dae" />
             </geometry>
         </collision>
@@ -132,5 +132,5 @@
             <origin xyz="${artag_x_pos} 0 ${hardware_z_offset}" rpy="-1.5707 0 1.5707" />
             <geometry>
-                <mesh filename="package://tec_proyect/meshes/aruco1.dae" />
+                <mesh filename="package://tec_proyect/meshes/aruco_id0.dae" />
             </geometry>
         </visual>

File: models/agv_model_three.urdf.xacro (robot description, xacro)
@@ -9,5 +9,5 @@
     <xacro:property name="chasis_length" value="${scale * 0.5}" />
     <xacro:property name="chasis_height" value="${scale * 0.3}" />
-    <xacro:property name="chasis_mass" value="${scale * 25}" />
+    <xacro:property name="chasis_mass" value="${scale * 150}" />
     <xacro:property name="base_x_offset" value="0.0" />
     <xacro:property name="chasis_x_pos" value="${base_x_offset/1.0}" />
@@ -37,5 +37,5 @@
     <xacro:property name="wheel_length" value="${scale * 0.05}" />
     <xacro:property name="wheel_radius" value="${scale * 0.08}" />
-    <xacro:property name="wheel_mass" value="${scale * 1.5}" />
+    <xacro:property name="wheel_mass" value="${scale * 2.637}" />
     <xacro:property name="wheel_x_offset" value="${base_x_offset + chasis_length/2.0}" />
     <xacro:property name="wheel_y_offset" value="${chasis_width/2.0 - wheel_length/2.0}" />
@@ -124,5 +124,5 @@
             <origin xyz="${artag_x_pos} 0 ${hardware_z_offset}" rpy="-1.5707 0 1.5707" />
             <geometry>
-                <mesh filename="package://tec_proyect/meshes/aruco3.dae" />
+                <mesh filename="package://tec_proyect/meshes/aruco_id2.dae" />
             </geometry>
         </collision>
@@ -130,5 +130,5 @@
             <origin xyz="${artag_x_pos} 0 ${hardware_z_offset}" rpy="-1.5707 0 1.5707" />
             <geometry>
-                <mesh filename="package://tec_proyect/meshes/aruco3.dae" />
+                <mesh filename="package://tec_proyect/meshes/aruco_id2.dae" />
             </geometry>
         </visual>

File: models/agv_model_two.urdf.xacro (robot description, xacro)
@@ -9,5 +9,5 @@
     <xacro:property name="chasis_length" value="${scale * 0.5}" />
     <xacro:property name="chasis_height" value="${scale * 0.3}" />
-    <xacro:property name="chasis_mass" value="${scale * 25}" />
+    <xacro:property name="chasis_mass" value="${scale * 150}" />
     <xacro:property name="base_x_offset" value="0.0" />
     <xacro:property name="chasis_x_pos" value="${base_x_offset/1.0}" />
@@ -37,5 +37,5 @@
     <xacro:property name="wheel_length" value="${scale * 0.05}" />
     <xacro:property name="wheel_radius" value="${scale * 0.08}" />
-    <xacro:property name="wheel_mass" value="${scale * 1.5}" />
+    <xacro:property name="wheel_mass" value="${scale * 2.637}" />
     <xacro:property name="wheel_x_offset" value="${base_x_offset + chasis_length/2.0}" />
     <xacro:property name="wheel_y_offset" value="${chasis_width/2.0 - wheel_length/2.0}" />
@@ -124,5 +124,5 @@
             <origin xyz="${artag_x_pos} 0 ${hardware_z_offset}" rpy="-1.5707 0 1.5707" />
             <geometry>
-                <mesh filename="package://tec_proyect/meshes/aruco2.dae" />
+                <mesh filename="package://tec_proyect/meshes/aruco_id1.dae" />
             </geometry>
         </collision>
@@ -130,5 +130,5 @@
             <origin xyz="${artag_x_pos} 0 ${hardware_z_offset}" rpy="-1.5707 0 1.5707" />
             <geometry>
-                <mesh filename="package://tec_proyect/meshes/aruco2.dae" />
+                <mesh filename="package://tec_proyect/meshes/aruco_id1.dae" />
             </geometry>
         </visual>

Commit message: First Commit

File: models/agv_macros.xacro (robot description, xacro)
@@ -7,7 +7,10 @@
                 <origin xyz = "0 0 0" rpy="0 1.5707 1.5707" />
                 <mass value="${mass}"/>
-                <inertia ixx="${mass * (3*radius*radius+(leng*leng))/12}" ixy="0" ixz="0"
-                         iyy = "${mass * (3*radius*radius+(leng*leng))/12}" iyz="0"
-                         izz = "${mass * (radius*radius)/2}" />
+<!--                <inertia ixx="${mass * (3*radius*radius+(leng*leng))/12}" ixy="0" ixz="0"-->
+<!--                         iyy = "${mass * (3*radius*radius+(leng*leng))/12}" iyz="0" -->
+<!--                         izz = "${mass * (radius*radius)/2}" />-->
+                <inertia ixx = "1e-3"    ixy="0" ixz="0"
+                         iyy = "1e-3"   iyz="0"
+                         izz = "1e-3" />
             </inertial>
             <visual>
@@ -26,12 +29,12 @@
                     <friction>
                         <kp>1000000.0</kp> <!-- kp and kd for rubber -->
-                        <kd>1.0</kd>
-                        <mu1>1.0</mu1>    <!-- Coulomb friction mus-->
-                        <mu2>1.0</mu2>  <!-- Friction coefficient muk-->
+                        <kd>100.0</kd>
+                        <mu1>1.0</mu1>      <!-- Coulomb friction mus-->
+                        <mu2>1.0</mu2>      <!-- Friction coefficient muk-->
                         <fdir1>1 0 0</fdir1>
-                        <slip1>0.0</slip1>
+                        <slip1>0.5</slip1>
                         <slip2>0.0</slip2>
-                        <maxVel>10.0</maxVel>
-                        <minDepth>0.001</minDepth>
+<!--                        <maxVel>1.0</maxVel>-->
+<!--                        <minDepth>0.001</minDepth>-->
                     </friction>
                 </surface>
@@ -43,7 +46,78 @@
             <parent link="${parent}"/>
             <axis xyz="0 1 0" rpy="0 0 0"/>
-            <limit effort="100" velocity="5.0"/>
-            <joint_properties damping="0.7"/>
+            <anchor xyz="0 0 0"/>
+            <limit effort="10000" velocity="1000"/>
+            <joint_properties damping="1.0" friction="1.0"/>
         </joint>
     </xacro:macro>
+    <!-- ************************ Create MaxBotix Sonar EZ4 ************************ -->
+    <xacro:macro name="sonar_sensor" params="name parent *origin ros_topic update_rate min_range max_range field_of_view ray_count">
+        <link name="${name}_link">
+            <inertial>
+                <mass value="0.001" />
+                <origin xyz="0 0 0" rpy="0 0 0" />
+                <inertia ixx="0.000000017" ixy="0" ixz="0" iyy="0.000000017" iyz="0" izz="0.000000017" />
+            </inertial>
+            <visual>
+                <origin xyz="0 0 0" rpy="0 0 0" />
+                <geometry>
+                    <mesh filename="package://tec_proyect/meshes/max_sonar_ez4.dae"/>
+                </geometry>
+            </visual>
+            <collision>
+                <origin xyz="0 0 0" rpy="0 0 0" />
+                <geometry>
+                    <box size="0.01 0.01 0.01" />
+                </geometry>
+            </collision>
+        </link>
+        <joint name="${name}_sonar_joint" type="fixed">
+            <xacro:insert_block name="origin" />
+            <child link="${name}_link"/>
+            <parent link="${parent}"/>
+        </joint>
+        <gazebo reference="${name}_link">
+          <sensor type="ray" name="${name}">
+            <always_on>true</always_on>
+            <update_rate>${update_rate}</update_rate>
+            <pose>0 0 0 0 0 0</pose>
+            <visualize>false</visualize>
+            <ray>
+              <scan>
+                <horizontal>
+                  <samples>${ray_count}</samples>
+                  <resolution>1</resolution>
+                  <min_angle>-${field_of_view/2}</min_angle>
+                  <max_angle> ${field_of_view/2}</max_angle>
+                </horizontal>
+                <vertical>
+                  <samples>${ray_count}</samples>
+                  <resolution>1</resolution>
+                  <min_angle>-${field_of_view/2}</min_angle>
+                  <max_angle> ${field_of_view/2}</max_angle>
+                </vertical>
+              </scan>
+              <range>
+                <min>${min_range}</min>
+                <max>${max_range}</max>
+                <resolution>0.01</resolution>
+              </range>
+                <noise>
+                    <type>gaussian</type>
+                    <!-- Noise parameters based on published spec for Hokuyo laser
+                    achieving "+-30mm" accuracy at range < 10m.  A mean of 0.0m and
+                    stddev of 0.01m will put 99.7% of samples within 0.03m of the true
+                    reading. -->
+                    <mean>0.0</mean>
+                    <stddev>0.01</stddev>
+                </noise>
+            </ray>
+            <plugin name="gazebo_ros_${name}_controller" filename="libhector_gazebo_ros_sonar.so">
+              <gaussianNoise>0.005</gaussianNoise>
+              <topicName>${ros_topic}</topicName>
+              <frameId>${name}_link</frameId>
+            </plugin>
+          </sensor>
+        </gazebo>
+    </xacro:macro>
 </robot>

File: models/agv_model.urdf.xacro (robot description, xacro)
@@ -6,6 +6,6 @@
     <xacro:property name="scale" value="1.0" />
     <!-- Length along X-axis, Width along Y-axis, Height along Z-axis -->
-    <xacro:property name="chasis_width" value="${scale * 0.5}" />
-    <xacro:property name="chasis_length" value="${scale * 0.5}" />
+    <xacro:property name="chasis_width" value="${scale * 0.46}" />
+    <xacro:property name="chasis_length" value="${scale * 0.46}" />
     <xacro:property name="chasis_height" value="${scale * 0.3}" />
     <xacro:property name="chasis_mass" value="${scale * 150}" />
